File: sch/usb-killer-detector.kicad_pcb (KiCad board)
At the start: 2 copper layers, 44 x 82 mm, 35 parts, among them J1 USB_A, J2 USB_C_Receptacle_PowerOnly_6P, Q2 2N3904, U1 LM339

Commit message: PCB: GND
Routing:
- net Net-(D5-K): track 11.0 -> 46.3 mm, vias 0 -> 1
- added copper zone on B.Cu, net GND
- added copper zone on F.Cu, net GND
Changed lines of the file:
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@@
+		(net "Net-(D5-K)")
+	)
+	(via
+		(at 100.225 108.56)
+		(size 0.6)
+		(drill 0.3)
+		(layers "F.Cu" "B.Cu")
+		(net "Net-(D5-K)")
+	)
+	(segment
+		(start 83.5 94.04)
+		(end 82.4 92.94)
+		(width 0.2)
+		(layer "B.Cu")
+		(net "Net-(D5-K)")
+	)
+	(segment
+		(start 100.225 98.186497)
+		(end 100.225 108.56)
+		(width 0.2)
+		(layer "B.Cu")
+		(net "Net-(D5-K)")
+	)
+	(segment
+		(start 92.438503 90.4)
+		(end 100.225 98.186497)
+		(width 0.2)
+		(layer "B.Cu")
+		(net "Net-(D5-K)")
+	)
+	(segment
+		(start 82.4 92.94)
+		(end 82.4 90.715256)
+		(width 0.2)
+		(layer "B.Cu")
+		(net "Net-(D5-K)")
+	)
+	(segment
+		(start 82.4 90.715256)
+		(end 82.715256 90.4)
+		(width 0.2)
+		(layer "B.Cu")
+		(net "Net-(D5-K)")
+	)
+	(segment
+		(start 82.715256 90.4)
+		(end 92.438503 90.4)
+		(width 0.2)
+		(layer "B.Cu")
 		(net "Net-(D5-K)")
 	)
@@
 	)
 	(segment
+		(start 84.5 66.5)
+		(end 85.23 65.77)
+		(width 0.2)
+		(layer "F.Cu")
+		(net "5V")
+	)
+	(segment
 		(start 77 90.5)
 		(end 77.42 90.5)
@@
 	)
 	(segment
+		(start 68.5 73)
+		(end 75 66.5)
+		(width 0.2)
+		(layer "F.Cu")
+		(net "5V")
+	)
+	(segment
 		(start 85.23 65.77)
 		(end 85.23 65.12)
@@
 	)
 	(segment
-		(start 75.5 66)
-		(end 85 66)
-		(width 0.2)
-		(layer "F.Cu")
-		(net "5V")
-	)
-	(segment
-		(start 68.5 73)
-		(end 75.5 66)
-		(width 0.2)
-		(layer "F.Cu")
-		(net "5V")
-	)
-	(segment
 		(start 97 127.5)
 		(end 102 127.5)
@@
 	)
 	(segment
-		(start 85 66)
-		(end 85.23 65.77)
-		(width 0.2)
-		(layer "F.Cu")
-		(net "5V")
-	)
-	(segment
 		(start 80.71 93.79)
 		(end 83.5 96.58)
@@
 		(start 97 117.38)
 		(end 97 127.5)
+		(width 0.2)
+		(layer "F.Cu")
+		(net "5V")
+	)
+	(segment
+		(start 75 66.5)
+		(end 84.5 66.5)
 		(width 0.2)
 		(layer "F.Cu")
@@
 		(net "Net-(D13-K)")
 	)
+	(zone
+		(net "GND")
+		(layers "F.Cu" "B.Cu")
+		(name "GND")
+		(hatch edge 0.5)
+		(connect_pads yes
+			(clearance 0.5)
+		)
+		(min_thickness 0.25)
+		(fill yes
+			(thermal_gap 0.5)
+			(thermal_bridge_width 0.5)
+			(island_removal_mode 1)
+		)
+		(polygon
+			(pts
+				(xy 59.5 47) (xy 121 47.5) (xy 119.5 151) (xy 60.5 151.5)
+			)
+		)
+	)
 	(embedded_fonts no)
