File: sch/usb-killer-detector.kicad_sch (KiCad schematic)
At the start: 35 parts, among them J1 USB_A, J2 USB_C_Receptacle_PowerOnly_6P, Q2 2N3904, U1 LM339

Commit message: Reprise v2 : schéma refait, PCB routé et dossier de fabrication
- Détection des deux polarités sur D+, D- et VBUS : comparateurs à
  fenêtre (2x LM339), seuils D+/D- +6,2 V / -5,0 V, VBUS +6,3 V / -0,3 V
- Alerte mémorisée (74HC279) avec bouton RESET et reset à la mise
  sous tension ; LED verte « OK » quand aucune alerte
- Protections : TVS SMAJ5.0A, clamps BAT54S, diode anti-retour SS34,
  polyfuse 500 mA
- PCB 44 x 82 mm entièrement routé, plans de masse sur les deux faces
- Règles d'isolation des lignes haute tension (kicad_dru) et classes
  de pistes (Power, HV)
- ERC 0, DRC 0 : les 2 avertissements de sérigraphie du connecteur
  USB-A (corps hors carte par construction) sont exclus avec justification
- sch/fabrication : Gerber + perçage (zip prêt à envoyer), BOM,
  fichier de placement, schéma et plan d'assemblage en PDF
- .gitignore : historique local de KiCad 10 (.history/)

Co-Authored-By: Claude Opus 5.5 <noreply@anthropic.com>
Parts:
- removed D1, D14, D15: D_Schottky, Diode_THT:D_DO-201AD_P15.24mm_Horizontal, symbol Device:D_Schottky
- removed D10, D4, D7: PTVS7V5Z1USK, Diode_SMD:Nexperia_DSN1608-2_1.6x0.8mm, symbol Diode:PTVS7V5Z1USK
- removed D12, D5, D9: PTVS7V5Z1USK, Diode_SMD:D_01005_0402Metric, symbol Diode:PTVS7V5Z1USK
- removed D13: LED_G, LED_THT:LED_D5.0mm, symbol Device:LED
- removed D16: LED_O, LED_THT:LED_D5.0mm, symbol Device:LED
- removed D6: LED_R_D+, LED_THT:LED_D5.0mm, symbol Device:LED
- removed D8: LED_R_D-, LED_THT:LED_D5.0mm, symbol Device:LED
- removed Q2: 2N3904, Package_TO_SOT_THT:TO-92_Inline, symbol Transistor_BJT:2N3904
- added C1: 10uF, Capacitor_SMD:C_0805_2012Metric, symbol Device:C
- added C10, C2, C3, C4, C8, C9: 100nF, Capacitor_SMD:C_0805_2012Metric, symbol Device:C
- added C11: 1uF, Capacitor_SMD:C_0805_2012Metric, symbol Device:C
- added C5, C6, C7: 1nF, Capacitor_SMD:C_0805_2012Metric, symbol Device:C
- added D1, D4: SMAJ5.0A, Diode_SMD:D_SMA, symbol Diode:SMAJ5.0A
- added D10: Rouge D-, LED_THT:LED_D5.0mm, symbol Device:LED
- added D12, D13, D14, D8: 1N4148W, Diode_SMD:D_SOD-123, symbol Diode:1N4148W
- added D15: Verte OK, LED_THT:LED_D5.0mm, symbol Device:LED
- added D2: Orange PWR, LED_THT:LED_D5.0mm, symbol Device:LED
- added D3: SS34, Diode_SMD:D_SMA, symbol Diode:SS34
- added D5, D6, D7: BAT54S, Package_TO_SOT_SMD:SOT-23, symbol Diode:BAT54S
- added D9: Rouge D+, LED_THT:LED_D5.0mm, symbol Device:LED
- added R17: 43k, Resistor_SMD:R_0805_2012Metric, symbol Device:R
- added R18, R19, R20: 10k, Resistor_SMD:R_0805_2012Metric, symbol Device:R
- added R21, R25: 100k, Resistor_SMD:R_0805_2012Metric, symbol Device:R
- added R22, R23, R24, R26: 1k, Resistor_SMD:R_0805_2012Metric, symbol Device:R
- added SW1: RESET, Button_Switch_SMD:SW_SPST_B3S-1000, symbol Switch:SW_Push
- added unit 4 of U1
- added U2: LM339, Package_SO:SOIC-14_3.9x8.7mm_P1.27mm, symbol Comparator:LM339
- added U3: 74HC279, Package_SO:SOIC-16_3.9x9.9mm_P1.27mm, symbol 74xx:74LS279
- D11: value LED_R_D- -> Rouge VBUS
- F1: value Polyfuse 250-500mA -> 500mA hold; footprint Fuse:Fuse_Bourns_MF-RG300 -> Fuse:Fuse_1812_4532Metric; MPN (none) -> Bourns MF-MSMF050-2
- J1: value USB_A -> USB-A test; MPN (none) -> GCT USB1046
- J2: value USB_C_Receptacle_PowerOnly_6P -> USB-C alim; footprint Connector_USB:USB_C_Receptacle_HRO_TYPE-C-31-M-12 -> Connector_USB:USB_C_Receptacle_GCT_USB4125-xx-x_6P_TopMnt_Horizontal; MPN (none) -> GCT USB4125-GF-A
- R1: value 1K -> 5.1k; footprint Resistor_THT:R_Axial_DIN0207_L6.3mm_D2.5mm_P7.62mm_Horizontal -> Resistor_SMD:R_0805_2012Metric
- R10: value 22K -> 120k; footprint Resistor_THT:R_Axial_DIN0207_L6.3mm_D2.5mm_P7.62mm_Horizontal -> Resistor_SMD:R_0805_2012Metric
- R11, R7: value 100K -> 220k; footprint Resistor_THT:R_Axial_DIN0207_L6.3mm_D2.5mm_P7.62mm_Horizontal -> Resistor_SMD:R_1206_3216Metric; Note (none) -> 1206, tenue HT
- R12: value 47K -> 220k; footprint Resistor_THT:R_Axial_DIN0207_L6.3mm_D2.5mm_P7.62mm_Horizontal -> Resistor_SMD:R_1206_3216Metric; Note (none) -> 1206, tenue HT
- R13: value 100K -> 220k; footprint Resistor_THT:R_Axial_DIN0207_L6.3mm_D2.5mm_P7.62mm_Horizontal -> Resistor_SMD:R_0805_2012Metric
- R14: value 5k -> 120k; footprint Resistor_THT:R_Axial_DIN0207_L6.3mm_D2.5mm_P7.62mm_Horizontal -> Resistor_SMD:R_0805_2012Metric
- R15: value 5k -> 100k; footprint Resistor_THT:R_Axial_DIN0207_L6.3mm_D2.5mm_P7.62mm_Horizontal -> Resistor_SMD:R_1206_3216Metric
- R16: value 10K -> 150k; footprint Resistor_THT:R_Axial_DIN0207_L6.3mm_D2.5mm_P7.62mm_Horizontal -> Resistor_SMD:R_0805_2012Metric
- R2: value 36K -> 5.1k; footprint Resistor_THT:R_Axial_DIN0207_L6.3mm_D2.5mm_P7.62mm_Horizontal -> Resistor_SMD:R_0805_2012Metric
- R3: value 10K -> 1k; footprint Resistor_THT:R_Axial_DIN0207_L6.3mm_D2.5mm_P7.62mm_Horizontal -> Resistor_SMD:R_0805_2012Metric
- R4: value 22 -> 51k; footprint Resistor_THT:R_Axial_DIN0207_L6.3mm_D2.5mm_P7.62mm_Horizontal -> Resistor_SMD:R_0805_2012Metric
- R5: value 100K -> 33k; footprint Resistor_THT:R_Axial_DIN0207_L6.3mm_D2.5mm_P7.62mm_Horizontal -> Resistor_SMD:R_0805_2012Metric
- R6: value 22K -> 15k; footprint Resistor_THT:R_Axial_DIN0207_L6.3mm_D2.5mm_P7.62mm_Horizontal -> Resistor_SMD:R_0805_2012Metric
- R8: value 22K -> 220k; footprint Resistor_THT:R_Axial_DIN0207_L6.3mm_D2.5mm_P7.62mm_Horizontal -> Resistor_SMD:R_1206_3216Metric; Note (none) -> 1206, tenue HT
- R9: value 390K -> 220k; footprint Resistor_THT:R_Axial_DIN0207_L6.3mm_D2.5mm_P7.62mm_Horizontal -> Resistor_SMD:R_0805_2012Metric
- U1: footprint Package_DIP:DIP-14_W7.62mm -> Package_SO:SOIC-14_3.9x8.7mm_P1.27mm; MPN (none) -> LM339DR
Connections:
- net GND: now also D11.1 (K), J1.SH (Shield), J2.SH (SHIELD), R1.2, R2.2, C1.2, C10.2, C11.2, C2.2, C3.2, C4.2, C5.2, C6.2, C7.2, C8.2, C9.2, D1.2 (A2), D10.1 (K), D2.1 (K), D4.2 (A2), D5.1 (A), D6.1 (A), D7.1 (A), D9.1 (K), R17.2, R25.2, SW1.2, U2.12 (V-), U2.8 (-), U3.14 (~{R}), U3.8 (GND); no longer R15.2, R3.2, R8.2
- net ALM_DM_N: now reaches U1.13
- net ALM_DM_N: now also R19.2, U1.14, U3.6 (~{S}); no longer D11.1 (K)
- net DM_HV: now reaches R11.2, R12.1
- net DP_HV: now reaches R7.2, R8.1
- net DP_HV: no longer U1.6 (-)
- net ALM_DP_N: now reaches U1.2
- net ALM_DP_N: now also U1.1, R18.2, U3.3 (~{S})
- net VL: now reaches R5.2, R6.1
- net VL: now also U1.6 (-), C4.1, U1.8 (-), U2.6 (-), U2.9 (+); no longer U1.4 (-)
- net X_DM: now reaches R13.2
- net X_DM: now also R12.2, R14.1, U1.10 (-), C6.1, D6.3 (COM), U1.9 (+)
- net X_DP: now reaches R10.1, R9.2
- net X_DP: now also R8.2, U1.4 (-), U1.7 (+), C5.1, D5.3 (COM); no longer U1.10 (-)
- net +5V: now reaches R4.1
- net +5V: now also J2.A9 (VBUS), J2.B9 (VBUS), R13.1, R16.1, R3.1, R9.1, U1.3 (V+), C1.1, C10.1, C2.1, C8.1, C9.1, D1.1 (A1), D3.2 (A), D5.2 (K), D6.2 (K), D7.2 (K), D8.1 (K), R18.1, R19.1, R20.1, R21.1, R26.1, U2.3 (V+), U3.11 (~{S}), U3.15 (~{S}), U3.16 (VCC), U3.2 (~{S}); no longer F1.2
- net CC1: now reaches J2.A5 (CC1)
- net CC1: now also R1.1; no longer R14.1
- net CC2: now reaches J2.B5 (CC2)
- net CC2: now also R2.1; no longer R15.1
- removed net 5V: D11.2 (A), J2.A9 (VBUS), J2.B9 (VBUS), R1.1, R11.1, R13.1, R16.2, R2.1, U1.3 (V+)
- net D+ renamed DP
- net DP: now also R7.1; no longer R5.1
- net D- renamed DM
- net DM: now also R11.1; no longer R7.1
- net VBUS renamed VBUS_PORT
- net VBUS_PORT: now also F1.2, R15.1, D4.1 (A1); no longer R4.2
- net VBUS_TEST renamed VBUS_SRC
- net VBUS_SRC: now also D3.1 (K); no longer R9.1
- removed net VREF: R2.2, R3.1, U1.11 (+), U1.5 (+), U1.7 (+)
- new net ALM_VBUS_N: R20.2, U2.1, U2.2, U3.12 (~{S})
- new net ANY_ALM: D12.1 (K), D13.1 (K), D14.1 (K), R25.1, U2.11 (+)
- new net LED_DM: D10.2 (A), R23.2
- new net LED_DP: D9.2 (A), R22.2
- new net LED_OK_A: D15.2 (A), R26.2
- new net LED_OK_K: D15.1 (K), U2.13
- new net LED_PWR: D2.2 (A), R3.2
- new net LED_VBUS: D11.2 (A), R24.2
- new net Q_DM: D13.2 (A), R23.1, U3.7 (Q)
- new net Q_DP: D12.2 (A), R22.1, U3.4 (Q)
- new net Q_VBUS: D14.2 (A), R24.1, U3.9 (Q)
- new net RST_N: C11.1, D8.2 (A), R21.2, SW1.1, U3.1 (~{R}), U3.10 (~{R}), U3.5 (~{R})
- new net VH: C3.1, R4.2, R5.1, U1.11 (+), U1.5 (+), U2.10 (-), U2.5 (+)
- new net X_VBUS: C7.1, D7.3 (COM), R15.2, R16.2, R17.1, U2.4 (-), U2.7 (+)
- no-connect marks 0 -> 2
Other:
- note added: "A. Alimentation USB-C (5 V)"
- note added: "Alarme mémorisée jusqu'au RESET (SW1) ou au débranchement de l'alim (R21/C11/D8)."
- note added: "B. Port sous test USB-A et protection VBUS"
- note added: "C. Références de seuil VH / VL"
- note added: "D. Étages d'entrée (fenêtre ±)"
- note added: "D3 empêche tout retour de tension vers le 5 V. D4 écrête VBUS vers +9 V / -1 V ; F1 coupe en cas de surcharge."
- note added: "E. Comparateurs LM339 (sorties collecteur ouvert)"
- note added: "Entrées D+/D- : 2 x 220k en 1206 (tenue >= 400 V). PCB : isolation >= 1 mm jusqu'à R8/R12."
- note added: "F. Mémoire d'alarme 74HC279"
- note added: "G. Voyants"
- note added: "H. Découplage, pull-ups, reset"
- note added: "LED rouge = alarme mémorisée sur la ligne ; LED verte = aucune alarme."
- note added: "Seuils d'alarme : D+ et D- au-dessus de +6,2 V ou en dessous de -5,0 V ; VBUS au-dessus de +6,3 V ou en dessous de -0,3 V. Seuils ratiométriques au 5 V (VH = 2,42 V, VL = 0,76 V)."
- note added: "VH = 5 V x 48/99 = 2,42 V VL = 5 V x 15/99 = 0,76 V"
- title: (none) -> SENTINELLE - Détecteur USB Killer
